File: Eagle/IPNS_v0.1/IPNS_v0.1.sch (EAGLE design)
At the start: 30 parts, among them J1 SWIM, J2 NFC, J3 BATT, J4 LEFT CONN, J5 RIGHT CONN, Q1 16MHz, Q2 32.768 kHz, U1 STM8L152C4_C6TX

Commit message: Board and schematic overall finished for MCU module. Need to check RC values
Other:
- note added: "Connectors: - SWIM - NFC Memory - Battery - Stimulator Circuit + Supply"
- note removed: "C5 and C8 Tantalum?"
- note removed: "STILL NEED TO IMPLEMENT: - MCU POWER SUPPLY - STIMULATOR CIRCUIT - STIMULATOR SUPPLY - VERIFY VALUES FOR MCU CONNECTIONS"
- note removed: "U2 IS INDUCTOR OR SHORT"
Changed lines of the file:
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@@
 </variantdefs>
 <classes>
-<class number="0" name="default" width="0.1778" drill="0.3048">
-<clearance class="0" value="0.2032"/>
+<class number="0" name="default" width="0.1524" drill="0.3048">
+<clearance class="0" value="0.1524"/>
 </class>
 </classes>
@@
 <sheet>
 <plain>
-<text x="66.04" y="124.46" size="1.778" layer="91">U2 IS INDUCTOR OR SHORT</text>
-<text x="66.04" y="129.54" size="1.778" layer="91">C5 and C8 Tantalum?</text>
-<text x="-7.62" y="132.08" size="1.778" layer="91">STILL NEED TO IMPLEMENT:
-- MCU POWER SUPPLY
-- STIMULATOR CIRCUIT
-- STIMULATOR SUPPLY
-- VERIFY VALUES FOR MCU CONNECTIONS</text>
+<text x="-45.72" y="132.08" size="1.778" layer="91">Connectors:
+- SWIM
+- NFC Memory
+- Battery
+- Stimulator Circuit + Supply</text>
 </plain>
 <instances>

Commit message: Made names font smaller; renumbered parts
Parts:
- removed R6, R7: 1k, IPNS_Lib_v0.1:R-US_R0805
- removed U$3: SLIDE_SWITCH, IPNS_Lib_v0.1:SLIDE_SWITCH
- added R1: 660, IPNS_Lib_v0.1:R-US_R0805
- added R2: 330, IPNS_Lib_v0.1:R-US_R0805
- added U$2: PUSH-BUTTON, IPNS_Lib_v0.1:PUSH-BUTTON
- C1, C8: value 1u -> 100n
- C10: value 7pF -> 20pF
- C12: value 1u -> 7pF
- C2: value 20pF -> 1u
- C3: value 20pF -> 100n
- C4: value 100n -> 20pF
- C6, C9: value 100n -> 1u
- J4: value LEFT CONN -> RIGHT CONN
- J5: value RIGHT CONN -> LEFT CONN
- LED1: value RED -> BLUE
- LED3: value BLUE -> RED
- R3: value 220 -> 1k
- R4: value 330 -> 1k
- R5: value 660 -> 220
- U$1: value PUSH-BUTTON -> SLIDE_SWITCH; device IPNS_Lib_v0.1:PUSH-BUTTON -> IPNS_Lib_v0.1:SLIDE_SWITCH
Connections:
- removed net N$11 (its old number): LED1.A, R3.1
- new net N$13: LED1.A, R1.1
- net +3V3: now also C2.1, C3.1, C9.2, J4.2, R4.2, R5.2, U$1.OUT2; no longer C1.1, C12.2, C9.1, J5.2, R6.2, R7.2, U$3.OUT2
- net DAC: now also J5.3; no longer J4.3
- net GND: now also C2.2, C3.2, C4.1, C9.1, U$2.P$1; no longer C2.1, C3.1, C4.2, C9.2, U$1.P$1
- net N$1: now also C10.2; no longer C2.2
- net N$12: now also R2.1; no longer R4.1
- net N$5: now also C4.2; no longer C3.2
- net N$6: now also C12.2; no longer C10.2
- net PWM: now also J5.4; no longer J4.4
- net RESET: now also C1.1, U$2.P$2; no longer C4.1, U$1.P$2
- net SCL: now also R3.1; no longer R6.1
- net SDA: now also R4.1; no longer R7.1
- net VBATT: now also J5.2, U$1.IN; no longer J4.2, U$3.IN
- net VLED2: now also R2.2; no longer R4.2
- net VLED3: now also R1.2; no longer R5.2
Other:
- moved on the sheet: C1, C10, C12, C2, C3, C4, C5, C6, C7, C8, C9, J4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
