File: Eagle/IPNS_v0.1/IPNS_v0.1 STIM.sch (EAGLE design)
At the start: 0 parts

Commit message: Developed a CAD model for the mosfet part
Parts:
- added C1, C2, C3: (no value), IPNS_Lib_v0.1:C-USC0805
- added M1, M2: DMN1019UVT, IPNS_Lib_v0.1:DMN1019UVT
- added R1, R2, R3, R4: (no value), IPNS_Lib_v0.1:R-US_R0805
- added U1: LTC3459ES6TRMPBF, IPNS_Lib_v0.1:LTC3459ES6TRMPBF
- added U2: LT1492CS8TRPBF, IPNS_Lib_v0.1:LT1492CS8TRPBF
