File: Eagle/IPNS_v0.1/IPNS_v0.1 MCU.brd (EAGLE design)
At the start: 32.9 x 33 mm, 30 parts, among them J1 SWIM, J2 NFC, J3 BATT, J4 RIGHT CONN, J5 LEFT CONN, Q1 16MHz, Q2 32.768 kHz, U1 STM8L152C4_C6TX

Commit message: Started IPNS_v0.2
Parts:
- R5: value 220 -> 1k
Changed lines of the file:
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@@
 <attribute name="NAME" x="4.826" y="25.908" size="0.6096" layer="25" rot="R90"/>
 </element>
-<element name="R5" library="IPNS_Lib_v0.1" package="R0805" value="220" x="18.288" y="30.48" smashed="yes">
+<element name="R5" library="IPNS_Lib_v0.1" package="R0805" value="1k" x="18.288" y="30.48" smashed="yes">
 <attribute name="NAME" x="19.685" y="28.194" size="0.6096" layer="25" rot="R90"/>
 </element>
