File: Eagle/IPNS_v0.1/IPNS_v0.1 MCU.sch (EAGLE design)
At the start: 30 parts, among them J1 SWIM, J2 NFC, J3 BATT, J4 RIGHT CONN, J5 LEFT CONN, Q1 16MHz, Q2 32.768 kHz, U1 STM8L152C4_C6TX

Commit message: Started IPNS_v0.2
Parts:
- R5: value 220 -> 1k
Changed lines of the file:
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@@
 <part name="C11" library="IPNS_Lib_v0.1" deviceset="C-US" device="C0805" value="7pF"/>
 <part name="GND5" library="IPNS_Lib_v0.1" deviceset="GND" device=""/>
-<part name="R5" library="IPNS_Lib_v0.1" deviceset="R-US_" device="R0805" value="220"/>
+<part name="R5" library="IPNS_Lib_v0.1" deviceset="R-US_" device="R0805" value="1k"/>
 <part name="R2" library="IPNS_Lib_v0.1" deviceset="R-US_" device="R0805" value="330"/>
 <part name="R1" library="IPNS_Lib_v0.1" deviceset="R-US_" device="R0805" value="660"/>
