File: Eagle/IPNS_v0.2/IPNS_v0.2.brd (EAGLE design)
At the start: 32.9 x 33 mm, 30 parts, among them J1 SWIM, J2 NFC, J3 BATT, J4 RIGHT CONN, J5 LEFT CONN, Q1 16MHz, Q2 32.768 kHz, U1 STM8L152C4_C6TX

Commit message: Started IPNS_v0.2
Parts:
- added C13: 100pF, IPNS_Lib_v0.1:C0805
- added C14: 47pF, IPNS_Lib_v0.1:C0805
- added C15: 4.7uF, IPNS_Lib_v0.1:C0805
- added C16: 1u, IPNS_Lib_v0.1:C0805
- added J10, J9: (no value), IPNS_Lib_v0.1:1X06
- added J6: OUTPUT CONN, IPNS_Lib_v0.1:1X02
- added J7: POL SWITCH CONN, IPNS_Lib_v0.1:1X04
- added J8: (no value), IPNS_Lib_v0.1:1X02
- added L1: 33uH, IPNS_Lib_v0.1:L2012C
- added LED4: RED, IPNS_Lib_v0.1:CHIP-LED0805
- added R10: 1k, IPNS_Lib_v0.1:M0805
- added R6: 200, IPNS_Lib_v0.1:R0805
- added R7: 2Meg, IPNS_Lib_v0.1:R0805
- added R8: 280k, IPNS_Lib_v0.1:R0805
- added R9: 1k, IPNS_Lib_v0.1:R0805
- added U$3, U$4: DMN1019USN, IPNS_Lib_v0.1:DMN1019USN
- added U$5: SLIDE_SWITCH, IPNS_Lib_v0.1:SLIDE_SWITCH
- added U2: LTC3459ES6TRMPBF, IPNS_Lib_v0.1:TSOT-23_S6
- added U3: LT1492CS8TRPBF, IPNS_Lib_v0.1:SO-8_S
- R5: value 220 -> 1k
- moved C12 120.9 mm to (55.9, -81.3)
- moved LED3 120.4 mm to (29.2, -88.9), turned to 0 degrees
- moved R5 118.1 mm to (17.8, -87.6)
- moved C11 116.4 mm to (50.8, -81.3)
- moved R4 111.4 mm to (12.7, -87.6)
- moved R3 109.6 mm to (7.62, -87.6)
- moved C10 108.9 mm to (34.3, -81.3), turned to 0 degrees
- moved C9 108.1 mm to (2.54, -87.6), turned to 0 degrees
- moved C6 106.9 mm to (71.1, -81.3), turned to 0 degrees
- moved C5 104.8 mm to (66.0, -81.3)
- moved C2 103.3 mm to (61.0, -81.3), turned to 0 degrees
- moved C8 96.7 mm to (21.6, -81.3)
- moved LED1 95.8 mm to (22.9, -88.9), turned to 0 degrees
- moved R2 93.9 mm to (45.7, -81.3), turned to 0 degrees
- moved R1 93.5 mm to (40.6, -81.3), turned to 0 degrees
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Connections:
- new net N$10: J9.6
- new net N$2: C13.1, U$3.G, U3.1
- new net N$25: J9.5
- new net N$26: J9.4
- new net N$27: J9.3
- new net N$29: J10.5
- new net N$30: J10.6
- new net N$4: C13.2, R6.2, U$3.S, U3.2
- new net N$7: C14.1, R7.1, R8.2, U2.3
- new net N$8: L1.1, U2.1
- new net N$9: LED4.A, R10.2
- new net SHDN: J8.1, U2.4
- new net VBOOST: C14.2, C15.1, J7.2, R7.2, U2.5, U3.8
- new net VCASE: J6.2, J7.4
- new net VDAC: J10.3, U$4.D
- new net VELEC: J6.1, J7.3
- new net VIN: R9.2, U$4.S, U3.3
- new net VLOW: J7.1, U$3.D
- new net VON: C16.1, J8.2, L1.2, R10.1, U$5.4, U2.6
- new net VPWM: J10.4, U$4.G
- net +3V3: now also J9.2
- net GND: now also C15.2, C16.2, J10.1, J9.1, LED4.C, R6.1, R8.1, R9.1, U2.2, U3.4
- net VBATT: now also J10.2, U$5.3
Routing:
- net +3V3: track 51.0 -> 0.00 mm, vias 6 -> 0
- net VBATT: track 49.0 -> 0.00 mm, vias 1 -> 0
- net ST_LINK_SWIM: track 33.7 -> 0.00 mm, vias 1 -> 0
- net RESET: track 30.5 -> 0.00 mm, vias 2 -> 0
- net PD1: track 26.5 -> 0.00 mm, vias 1 -> 0
- net PD0: track 26.4 -> 0.00 mm, vias 1 -> 0
- net PWM: track 25.0 -> 0.00 mm, vias 1 -> 0
- net VREFINT: track 22.9 -> 0.00 mm, vias 1 -> 0
- net DAC: track 20.9 -> 0.00 mm, vias 1 -> 0
- net PC4: track 20.3 -> 0.00 mm, vias 1 -> 0
- net N$5: track 14.1 -> 0.00 mm, vias 1 -> 0
- net SCL: track 13.4 -> 0.00 mm, vias 2 -> 0
- net VLED2: track 11.1 -> 0.00 mm
- net N$6: track 10.8 -> 0.00 mm
- net N$1: track 9.31 -> 0.00 mm
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- removed copper zone on layer 16, net +3V3
- removed copper zone on layer 1, net GND
Other:
- board size 32.9 x 33 mm -> 160 x 100 mm
- board text removed: "Alexey Revinski"
- board text removed: "IPNS_v0.1 MCU"
- board text removed: "NU BME 390"

Commit message: Fixed polarity switching inversion + initialization problems
Parts:
- removed J10, J9: (no value), IPNS_Lib_v0.1:1X06
- removed J2: NFC, IPNS_Lib_v0.1:1X04
- removed J5: LEFT CONN, IPNS_Lib_v0.1:1X12
- removed J7: POL SWITCH CONN, IPNS_Lib_v0.1:1X04
- removed J8: (no value), IPNS_Lib_v0.1:1X02
- removed LED3: RED, led:CHIP-LED0805
- removed LED4: RED, IPNS_Lib_v0.1:CHIP-LED0805
- removed R10: 1k, IPNS_Lib_v0.1:M0805
- added C17, C18: 4.7u, IPNS_Lib:C0603
- added U$6: MCP78381, IPNS_Lib:SOT23-5L
- added U4: STM8L151GXUX, IPNS_Lib:UFQFPN-28
- C1, C10, C11, C12, C13, C14, C15, C16, C2, C3, C4, C6, C7, C8, C9: device IPNS_Lib_v0.1:C0805 -> IPNS_Lib_v0.1:C0603
- C5: value 1u -> 100n; device IPNS_Lib_v0.1:C0805 -> IPNS_Lib_v0.1:C0603
- J4: value RIGHT CONN -> NFC; device IPNS_Lib_v0.1:1X12 -> IPNS_Lib_v0.1:1X04
- L1: device IPNS_Lib_v0.1:L2012C -> IPNS_Lib_v0.1:L0201
- LED1: value BLUE -> RED; device led:CHIP-LED0805 -> IPNS_Lib:SML0603
- LED2: device led:CHIP-LED0805 -> IPNS_Lib:SML0603
- R1: value 660 -> 1k; device IPNS_Lib_v0.1:R0805 -> IPNS_Lib:R0603
- R2: value 330 -> 1k; device IPNS_Lib_v0.1:R0805 -> IPNS_Lib:R0603
- R3, R4: value 1k -> 4.7k; device IPNS_Lib_v0.1:R0805 -> IPNS_Lib_v0.1:R0603
- R5: value 1k -> 27k; device IPNS_Lib_v0.1:R0805 -> IPNS_Lib:R0603
- R6, R7, R8, R9: device IPNS_Lib_v0.1:R0805 -> IPNS_Lib_v0.1:R0603
- U$1: value SLIDE_SWITCH -> DMN1019USN; device IPNS_Lib_v0.1:SLIDE_SWITCH -> IPNS_Lib:DMN1019USN
- U$3: device IPNS_Lib_v0.1:DMN1019USN -> IPNS_Lib:DMN1019USN
- U$4: value DMN1019USN -> ISL60002; device IPNS_Lib_v0.1:DMN1019USN -> IPNS_Lib:ISL60002
- moved LED2 209.2 mm to (2.54, -262.9)
- moved J4 205.4 mm to (10.2, -214.6)
- moved R2 195.3 mm to (2.54, -271.8)
- moved R5 189.8 mm to (2.54, -276.9)
- moved R1 189.3 mm to (2.54, -266.7)
- moved C6 177.6 mm to (2.54, -245.1)
- moved LED1 171.4 mm to (2.54, -259.1)
- moved C5 171.0 mm to (2.54, -240.0)
- moved U$1 157.8 mm to (3.81, -226.1)
- moved U1 82.4 mm to (25.4, 12.7)
- moved U$4 66.0 mm to (3.81, -236.2)
- moved U$3 57.8 mm to (3.81, -229.9)
Connections:
- net ST_LINK_SWIM renamed SWIM
- removed net DAC: J5.3, U1.32
- removed net N$11 (its old number): LED3.A, R5.1
- removed net N$12: LED2.A, R2.1
- removed net N$25: J9.5
- removed net N$26: J9.4
- removed net N$27: J9.3
- removed net N$29: J10.5
- removed net N$30: J10.6
- removed net N$9 (its old number): LED4.A, R10.2
- removed net PC4: J4.4, U1.43
- removed net PD0: J5.6, U1.20
- removed net PD1: J5.5, U1.21
- removed net PWM: J5.4, U1.22
- removed net VLED2: R2.2, U1.25
- removed net VLED3: R1.2, U1.24
- removed net VREFINT: J4.3, U1.41
- new net N$1: LED1.C, LED2.A, U$6.1
- new net N$13: R5.2, U$6.5
- new net VDD1/VDDA/VREF+: U4.7
- new net VPOL: U1.24
- new net VPOW: C17.1, R1.2, U$6.4
- new net VREF: C5.1, C6.1, U$4.2, U1.12
- new net VSS1/VSSA/VREF-: U4.6
- net +3V3: now also C9.1, U$4.1; no longer C5.1, C6.1, C9.2, J2.2, J9.2, R5.2, U$1.4, U1.12
- net GND: now also C17.2, C18.1, C9.2, R2.1, R5.1, U$4.3, U$6.2; no longer C9.1, J10.1, J2.1, J4.12, J5.1, J5.12, J9.1, LED1.C, LED2.C, LED3.C, LED4.C
- net N$10: now also LED2.C, R2.2; no longer J9.6
- net N$2: now also U$3.S; no longer U$3.G
- net N$4: now also U$3.G; no longer U$3.S
- net SCL: now also J4.3, R4.1; no longer J2.3, R3.1
- net SDA: now also J4.4, R3.1; no longer J2.4, R4.1
- net SHDN: no longer J8.1
- net VBATT: now also C18.2, U$6.3; no longer J10.2, J5.2, U$1.3
- net VBOOST: no longer J7.2
- net VCASE: no longer J7.4
- net VDAC: now also U$1.D, U1.32; no longer J10.3, U$4.D
- net VELEC: no longer J7.3
- net VIN: now also U$1.S; no longer U$4.S
- net VLOW: no longer J7.1
- net VON: no longer J8.2, R10.1
- net VPWM: now also U$1.G, U1.22; no longer J10.4, U$4.G

Commit message: Developed IPNS_v0.2 further
Parts:
- removed J6: OUTPUT CONN, IPNS_Lib_v0.1:1X02
- removed Q1: 16MHz, IPNS_Lib_v0.1:HC49/S
- removed Q2: 32.768 kHz, IPNS_Lib_v0.1:TC26H
- removed U4: STM8L151GXUX, IPNS_Lib:UFQFPN-28
- added C19: 10u, IPNS_Lib:C0603
- added C20, C22: 0.1u, rcl:C0603
- added C21: 22u, rcl:C0603
- added IC1: TPS61201, IPNS_Lib:S-PDSO-N10
- added J2: (no value), IPNS_Lib:1X02
- added L2: 2.2u, rcl:L2012C
- added R10: 1k, IPNS_Lib:R0603
- added R11: 220k, rcl:R0603
- added R12: 1.2Meg, rcl:R0603
- added R13: 2Meg, rcl:R0603
- added R14: 180k, rcl:R0603
- added U$7: 40_CRYSTAL_16M, IPNS_Lib:X4-SMD-3.2X2.5X0.7MM
- added U$8: 32.768_CRYSTAL, IPNS_Lib:X2-SMD-3.2X1.5X0.55MM
- L1: device IPNS_Lib_v0.1:L0201 -> IPNS_Lib_v0.1:L2012C
- U$5: value SLIDE_SWITCH -> ADG1636; device IPNS_Lib_v0.1:SLIDE_SWITCH -> IPNS_Lib:TSSOP16
- moved C18 323.8 mm to (59.2, 31.8)
- moved C17 322.1 mm to (59.9, 35.1), turned to 270 degrees
- moved R5 318.7 mm to (55.9, 37.3)
- moved R2 311.1 mm to (53.8, 35.1), turned to 90 degrees
- moved R1 309.3 mm to (59.4, 37.3), turned to 180 degrees
- moved LED2 302.6 mm to (55.4, 35.1), turned to 270 degrees
- moved LED1 296.5 mm to (54.6, 32.8), turned to 180 degrees
- moved U$6 291.3 mm to (57.7, 34.5)
- moved U$3 286.2 mm to (37.6, 54.4), turned to 90 degrees
- moved U$1 272.0 mm to (38.9, 43.7), turned to 180 degrees
- moved C6 265.7 mm to (47.8, 16.8)
- moved C5 259.4 mm to (48.8, 15.2)
- moved U$4 252.7 mm to (48.8, 12.4), turned to 270 degrees
- moved J4 244.9 mm to (33.0, 29.2)
- moved R6 221.9 mm to (40.9, 51.3), turned to 180 degrees
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Connections:
- net VPWM renamed VTIM
- removed net N$5: C4.2, Q1.1, U1.4
- removed net N$9: C10.2, Q1.2, U1.3
- removed net VCASE: J6.2
- removed net VDD1/VDDA/VREF+: U4.7
- removed net VLOW: U$3.D
- removed net VON: C16.1, L1.2, U$5.4, U2.6
- removed net VSS1/VSSA/VREF-: U4.6
- new net N$12: C13.2, U$3.G, U3.1
- new net N$14: IC1.3, L2.2
- new net N$16: IC1.10, R11.2, R12.1
- new net N$17: C20.1, IC1.1
- new net N$18: C22.2, IC1.7, R13.1, R14.2
- new net N$22: U$5.12, U$5.13, U$5.14, U$5.2
- new net OSC161: C4.1, U$7.3, U1.3
- new net OSC162: C10.2, U$7.1, U1.4
- new net VBODY: U$5.3
- new net VSINK: U$3.D, U$5.10, U$5.4
- net +3V3: now also C21.1, IC1.2, R10.2, R12.2
- net GND: now also C19.2, C20.2, C21.2, C4.2, IC1.4, IC1.9, IC1.PP, IC1.PP@1, IC1.PP@2, J2.2, R11.1, R14.1, U$5.5, U$5.6, U$7.2, U$7.4, U3.5; no longer C4.1
- net N$2: now also R6.2, U3.2; no longer U3.1
- net N$3: now also U$8.1; no longer Q2.2
- net N$4: now also U3.6, U3.7; no longer C13.2, R6.2, U$3.G, U3.2
- net N$6: now also U$8.2; no longer Q2.1
- net RESET: now also R10.1
- net VBATT: now also C16.1, C19.1, C22.1, IC1.5, IC1.6, IC1.8, L1.2, L2.1, R13.2, U2.6; no longer U$5.3
- net VELEC: now also U$5.11; no longer J6.1
- net VPOL: now also U$5.1, U$5.9
- net VPOW: now also J2.1
Routing:
- net VBATT: track 0.00 -> 35.5 mm, vias 0 -> 3
- net +3V3: track 0.00 -> 33.1 mm, vias 0 -> 7
- net VPOL: track 0.00 -> 29.5 mm, vias 0 -> 3
- net RESET: track 0.00 -> 23.5 mm, vias 0 -> 2
- net GND: track 0.00 -> 13.8 mm
- net N$11: track 0.00 -> 13.0 mm, vias 0 -> 2
- net SCL: track 0.00 -> 11.4 mm, vias 0 -> 2
- net VPOW: track 0.00 -> 9.76 mm
- net SDA: track 0.00 -> 9.05 mm
- net N$2: track 0.00 -> 8.01 mm
- net SWIM: track 0.00 -> 7.95 mm, vias 0 -> 1
- net N$18: track 0.00 -> 7.49 mm
- net N$22: track 0.00 -> 7.32 mm
- net VBOOST: track 0.00 -> 7.17 mm
- net VSINK: track 0.00 -> 6.56 mm
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- added copper zone on layer 16, net +3V3
- added copper zone on layer 1, net GND

Commit message: Updated IPNS_v0.2
Parts:
- removed C5, C7, C8: 100n, IPNS_Lib_v0.1:C0603
- removed C6, C9: 1u, IPNS_Lib_v0.1:C0603
- removed J2: (no value), IPNS_Lib:1X02
- removed J3: BATT, IPNS_Lib_v0.1:1X02
- removed R10: 1k, IPNS_Lib:R0603
- removed R11: 220k, rcl:R0603
- removed R12: 1.2Meg, rcl:R0603
- removed U1: STM8L152C4_C6TX, IPNS_Lib_v0.1:LQFP48-7X7MM
- added J5, J6: (no value), IPNS_Lib:1X12
- added U$10, U$9: SCREWTERMINAL, IPNS_Lib:SCREWTERMINAL
- added U4: STM8L151GXUX, IPNS_Lib:UFQFPN-28
- U$4: value ISL60002 -> SCREWTERMINAL; device IPNS_Lib:ISL60002 -> IPNS_Lib:SCREWTERMINAL
- moved U$2 60.5 mm to (41.1, 85.6), turned to 270 degrees
- moved C18 54.6 mm to (10.4, 7.11), turned to 270 degrees
- moved R1 54.3 mm to (17.3, 3.05), turned to 0 degrees
- moved LED2 54.3 mm to (12.4, 1.78), turned to 0 degrees
- moved R2 53.7 mm to (10.7, 3.05), turned to 0 degrees
- moved R13 53.2 mm to (7.11, 9.91)
- moved U$6 52.8 mm to (13.7, 5.33), turned to 270 degrees
- moved R14 51.4 mm to (4.83, 16.8), turned to 90 degrees
- moved C17 51.0 mm to (17.3, 7.11), turned to 90 degrees
- moved R5 50.8 mm to (14.5, 7.87)
- moved C22 49.9 mm to (9.40, 19.1), turned to 0 degrees
- moved LED1 49.9 mm to (15.5, 1.78), turned to 0 degrees
- moved C19 49.9 mm to (10.7, 9.91), turned to 0 degrees
- moved L2 49.1 mm to (9.91, 11.9)
- moved C16 47.1 mm to (14.5, 9.91)
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Connections:
- removed net N$16: IC1.10, R11.2, R12.1
- removed net N$3: C11.2, U$8.1, U1.45
- removed net N$6: C12.2, U$8.2, U1.44
- removed net OSC161: C4.1, U$7.3, U1.3
- removed net OSC162: C10.2, U$7.1, U1.4
- removed net SHDN: U2.4
- removed net VREF: C5.1, C6.1, U$4.2, U1.12
- new net OSCH1: C4.1, U$7.3, U4.3
- new net OSCH2: C10.2, U$7.1, U4.2
- new net OSCL1: C12.2, U$8.2, U4.26
- new net OSCL2: C11.2, U$8.1, U4.27
- net +3V3: now also IC1.10, U4.7; no longer C7.1, C8.1, C9.1, R10.2, R12.2, U$4.1, U1.10, U1.11, U1.13, U1.39
- net GND: now also U$10.2, U$4.2, U4.6; no longer C5.2, C6.2, C7.2, C8.2, C9.2, J2.2, J3.2, R11.1, U$4.3, U1.40, U1.9
- net RESET: now also U4.1; no longer R10.1, U1.2
- net SCL: now also U4.22; no longer U1.38
- net SDA: now also U4.21; no longer U1.37
- net SWIM: now also U4.28; no longer U1.1
- net VBATT: now also U$10.1, U2.4; no longer J3.1
- net VBODY: now also U$9.1
- net VDAC: now also U4.17; no longer U1.32
- net VELEC: now also U$9.2
- net VPOL: now also U4.12; no longer U1.24
- net VPOW: now also U$4.1; no longer J2.1
- net VTIM: now also U4.10; no longer U1.22
Routing:
- net +3V3: track 33.1 -> 13.8 mm, vias 7 -> 3
- net VBATT: track 35.5 -> 51.7 mm, vias 3 -> 7
- net VPOL: track 29.5 -> 14.0 mm, vias 3 -> 2
- net N$18: track 7.49 -> 22.9 mm, vias 0 -> 3
- net RESET: track 23.5 -> 11.2 mm, vias 2 -> 1
- net N$11: track 13.0 -> 1.34 mm, vias 2 -> 0
- net SCL: track 11.4 -> 0.00 mm, vias 2 -> 0
- net SDA: track 9.05 -> 0.00 mm
- net N$1: track 2.80 -> 11.5 mm, vias 0 -> 2
- net GND: track 13.8 -> 5.70 mm
- net VBOOST: track 7.17 -> 14.4 mm, vias 0 -> 3
- net OSCH1: track 0.00 -> 6.87 mm
- net OSC161: track 6.15 -> 0.00 mm
- net VREF: track 5.84 -> 0.00 mm
- net OSCL1: track 0.00 -> 5.60 mm
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